Commit message: 完成属性添加

File: install/robo_build/share/robo_build/urdf/ins_bot/actuator/ins_bot.urdf.xacro (robot description, xacro)
@@ -2,10 +2,10 @@
 <robot xmlns:xacro="http://www.ros.org/wiki/xacro" name="ins_bot">
   <!-- 执行器组件 -->
-  <xacro:include filename="$(find ins_bot_description)/urdf/ins_bot/actuato/rwheel.urdf.xacro"/>
-  <xacro:include filename="$(find ins_bot_description)/urdf/ins_bot/actuator/caster.urdf.xacro"/>
+  <xacro:include filename="$(find robo_build)/urdf/ins_bot/actuator/wheel.urdf.xacro"/>
+  <xacro:include filename="$(find robo_build)/urdf/ins_bot/actuator/caster.urdf.xacro"/>
   <!-- 执行器主动轮 + 从动轮 -->
-  <xacro:wheel wheel_name="left" xyz="0 0.10 -0.06"/>
-  <xacro:wheel wheel_name="right" xyz="0 -0.10 -0.06"/>
-  <xacro:caster caster_name="front" xyz="0.08 0.0 -0.076"/>
-  <xacro:caster caster_name="back" xyz="-0.08 0.0 -0.076"/>
+  <xacro:wheel_xacro wheel_name="left" xyz="0 0.10 -0.06"/>
+  <xacro:wheel_xacro wheel_name="right" xyz="0 -0.10 -0.06"/>
+  <xacro:caster_xacro caster_name="front" xyz="0.08 0.0 -0.076"/>
+  <xacro:caster_xacro caster_name="back" xyz="-0.08 0.0 -0.076"/>
 </robot>

File: install/robo_build/share/robo_build/urdf/ins_bot/actuator/wheel.urdf.xacro (robot description, xacro)
@@ -4,5 +4,5 @@
     <link name="${wheel_name}_wheel_link">
       <visual>
-        <origin xyz="0 0 0" rpy="1.5707 0 0"/>
+        <origin xyz="0 0 0" rpy="1.57079 0 0"/>
         <geometry>
           <cylinder length="0.04" radius="0.032"/>

File: install/robo_build/share/robo_build/urdf/ins_bot/base.urdf.xacro (robot description, xacro)
@@ -1,4 +1,5 @@
 <?xml version="1.0"?>
 <robot xmlns:xacro="http://www.ros.org/wiki/xacro">
+  <xacro:include filename="$(find robo_build)/urdf/ins_bot/common_inertia.xacro"/>
   <xacro:macro name="base_xacro" params="length radius">
     <link name="base_footprint"/>
@@ -6,5 +7,5 @@
       <parent link="base_footprint"/>
       <child link="base_link"/>
-      <origin xyz="0.0 0.0 ${length / 2.0 + 0.032 - 0.001}" rpy="0 0 0"/>
+      <origin xyz="0.0 0.0 ${length/2.0 + 0.032 - 0.001}" rpy="0 0 0"/>
     </joint>
     <link name="base_link">
@@ -18,4 +19,15 @@
         </material>
       </visual>
+      <!-- 添加碰撞属性 -->
+      <collision>
+        <origin xyz="0 0 0.0" rpy="0 0 0"/>
+        <geometry>
+          <cylinder length="${length}" radius="${radius}"/>
+        </geometry>
+        <material name="white">
+          <color rgba="1.0 1.0 1.0 0.5"/>
+        </material>
+      </collision>
+      <xacro:cylinder_inertia m ="1.0" r="${radius}" h="${length}"/>
     </link>
   </xacro:macro>

File: install/robo_build/share/robo_build/urdf/ins_bot/ins_bot.urdf.xacro (robot description, xacro)
@@ -6,4 +6,5 @@
   <xacro:include filename="$(find robo_build)/urdf/ins_bot/sensor/laser.urdf.xacro"/>
   <xacro:include filename="$(find robo_build)/urdf/ins_bot/sensor/camera.urdf.xacro"/>
+  <xacro:include filename="$(find robo_build)/urdf/ins_bot/actuator/ins_bot.urdf.xacro"/>
   <xacro:base_xacro length="0.12" radius="0.1"/> <!-- 传感器 -->
   <xacro:imu_xacro xyz="0 0 0.02"/>

File: install/robo_build/share/robo_build/urdf/ins_bot/sensor/imu.urdf.xacro (robot description, xacro)
@@ -10,5 +10,5 @@
         <material name="black">
           <color rgba="0 0 0 0.8"/>
-        </material>  <!-- Corrected: closed the <material> tag -->
+        </material>
       </visual>
     </link>
